File: hardware/kicad/I2C_knob.kicad_sch (KiCad schematic)
At the start: 12 parts, among them J1 JST 4 Pin Qwiic I2C Connector, J2 JST 4 Pin Qwiic I2C Connector, J3 noknok_FlashPads_I2C-module, SW1 RotaryEncoder_Switch, U1 CH32V003J4M6

Commit message: Knob V2: rename status LED resistor R5 -> R2, add BOM
R5 was renamed to R2 in KiCad (R2/R3 freed up by the removed pull-ups).
Docs updated to match; added the exported BOM (.xls).
Parts:
- renumbered R5 to R2
Changed lines of the file:
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@@
 		(in_pos_files yes)
 		(dnp no)
-		(property "Reference" "R5"
+		(property "Reference" "R2"
 			(at 202.184 84.328 90)
 			(show_name no)
@@
 			(project "I2C_knob"
 				(path "/89ac1937-28eb-4c0f-a201-5c0292dd68d3"
-					(reference "R5")
+					(reference "R2")
 					(unit 1)
 				)

Commit message: hardware: update schematic, rename BOM and schematic PDF, fix readme links
Other:
- note removed: "Specs: - I2C powered at 3.3V"
